Commit message: add new world and navigation goal

File: mcr_environments/mcr_gazebo_worlds/common/worlds/brsu-c025-sim.urdf.xacro (robot description, xacro)
@@ -20,4 +20,6 @@
 					1-19-20
 					1-21-22-23
+            platforms: 8, 15, 22, 23, 12, 16, 18
+            enable wall for closing arena: 4,5,11,12
 -->
 <robot name="brsu-c025-config2">
@@ -90,5 +92,5 @@
   	</link>
   	<joint name="join3" type="fixed">
-    		<origin xyz="-0.580 0.421 0" rpy="0 0 1.570796"/>
+    		<origin xyz="-0.230 0.421 0" rpy="0 0 1.570796"/>
     		<parent link="wall_2"/>
     		<child link="wall_3"/>
@@ -103,11 +105,11 @@
       			<origin xyz="0 0 0"/>
       			<geometry>
-					<box size="0.04 1.2 0.3" /> <!--wall 120, width = 4 cm, lenght = 120 cm, height = 30 cm-->
-      			</geometry>
-    		</visual>
-			<collision>
-      			<origin xyz="0 0 0"/>
-				<geometry>
-					<box size="0.04 1.2 0.3"/>
+					<box size="0.04 0.5 0.3" /> <!--wall 120, width = 4 cm, lenght = 120 cm, height = 30 cm-->
+      			</geometry>
+    		</visual>
+			<collision>
+      			<origin xyz="0 0 0"/>
+				<geometry>
+					<box size="0.04 0.5 0.3"/>
 				</geometry>
     		</collision>
@@ -264,5 +266,5 @@
   	</link>
   	<joint name="join10" type="fixed">
-			<origin xyz="-0.580 -0.421 0" rpy="0 0 1.570796"/>
+			<origin xyz="-0.230 -0.421 0" rpy="0 0 1.570796"/>
     		<parent link="wall_9"/>
     		<child link="wall_10"/>
@@ -277,11 +279,11 @@
       			<origin xyz="0 0 0"/>
       			<geometry>
-					<box size="0.04 1.2 0.3" /> <!--wall 120, width = 4 cm, lenght = 120 cm, height = 30 cm-->
-      			</geometry>
-    		</visual>
-			<collision>
-      			<origin xyz="0 0 0"/>
-				<geometry>
-					<box size="0.04 1.2 0.3"/>
+					<box size="0.04 0.5 0.3" /> <!--wall 120, width = 4 cm, lenght = 120 cm, height = 30 cm-->
+      			</geometry>
+    		</visual>
+			<collision>
+      			<origin xyz="0 0 0"/>
+				<geometry>
+					<box size="0.04 0.5 0.3"/>
 				</geometry>
     		</collision>
@@ -533,31 +535,7 @@
     		</collision>
   	</link>
-  	<joint name="join21" type="fixed">
-			<origin xyz="-1.912 0.057 0" rpy="0 0 0"/>
+  	  	<joint name="join21" type="fixed">
+			<origin xyz="-1.912 0.057 -0.1" rpy="0 0 0"/>
     		<parent link="wall_1"/>
-    		<child link="wall_21"/>
-  	</joint>
-  	<link name="wall_21">
-    		<inertial>
-      			<origin xyz="0 0 0" />
-      			<mass value="10.0" />
-      			<inertia  ixx="1.0" ixy="0.0"  ixz="0.0"  iyy="1.0"  iyz="0.0"  izz="1.0" />
-    		</inertial>
-    		<visual>
-      			<origin xyz="0 0 0"/>
-      			<geometry>
-					<box size="0.04 0.8 0.3" /> <!--wall 80, width = 4 cm, lenght = 80 cm, height = 30 cm-->
-      			</geometry>
-    		</visual>
-			<collision>
-      			<origin xyz="0 0 0"/>
-				<geometry>
-					<box size="0.04 0.8 0.3"/>
-				</geometry>
-    		</collision>
-  	</link>
-  	<joint name="join22" type="fixed">
-			<origin xyz="-0.251 0 -0.1" rpy="0 0 0"/>
-    		<parent link="wall_21"/>
     		<child link="wall_22"/>
   	</joint>
@@ -569,40 +547,40 @@
     		</inertial>
     		<visual>
-      			<origin xyz="0 0 0"/>
-      			<geometry>
-					<box size="0.46 0.8 0.1" /> <!--platform, width = 46 cm, lenght = 80 cm, height = 10 cm-->
-      			</geometry>
-    		</visual>
-			<collision>
-      			<origin xyz="0 0 0"/>
-				<geometry>
-					<box size="0.46 0.8 0.1"/>
-				</geometry>
-    		</collision>
-  	</link>
-  	<joint name="join23" type="fixed">
-			<origin xyz="0.502 0 0" rpy="0 0 0"/>
-    		<parent link="wall_22"/>
-    		<child link="wall_23"/>
-  	</joint>
-  	<link name="wall_23">
-    		<inertial>
-      			<origin xyz="0 0 0" />
-      			<mass value="10.0" />
-      			<inertia  ixx="1.0" ixy="0.0"  ixz="0.0"  iyy="1.0"  iyz="0.0"  izz="1.0" />
-    		</inertial>
-    		<visual>
-      			<origin xyz="0 0 0"/>
-      			<geometry>
-					<box size="0.46 0.8 0.1" /> <!--platform, width = 46 cm, lenght = 80 cm, height = 10 cm-->
-      			</geometry>
-    		</visual>
-			<collision>
-      			<origin xyz="0 0 0"/>
-				<geometry>
-					<box size="0.46 0.8 0.1"/>
-				</geometry>
-    		</collision>
-  	</link>
+      			<origin xyz="0 0 0"/> <!-- -0.2 if table exists, 0.0 if not-->
+      			<geometry>
+					<box size="0.46 0.46 0.1"/>
+                </geometry>
+    		</visual>
+			<collision>
+      			<origin xyz="0 0 0"/>
+				<geometry>
+					<box size="0.46 0.46 0.1"/>
+				</geometry>
+    		</collision>
+  	</link>
+	<joint name="join_object1" type="fixed">
+        <origin xyz="0.075 0.0 0.0" rpy="0 0 0"/> <!-- y=-0.2 if table exists, -0.4 if not-->
+        <parent link="wall_22"/>
+        <child link="object1"/>
+    </joint>
+    <link name="object1">
+        	<inertial>
+      			<origin xyz="0 0 0" />
+      			<mass value="10.0" />
+      			<inertia  ixx="1.0" ixy="0.0"  ixz="0.0"  iyy="1.0"  iyz="0.0"  izz="1.0" />
+    		</inertial>
+    		<visual>
+      			<origin xyz="0 0 0"/>
+      			<geometry>
+					<mesh filename="package://mcr_gazebo_objects/common/models/bunny/meshes/textured_bunny_ml.dae" scale="0.735095 0.735095 0.735095"/>
+      			</geometry>
+    		</visual>
+			<!--collision>
+      			<origin xyz="0 0 0"/>
+				<geometry>
+					<box size="0.46 0.46 0.0"/>
+				</geometry>
+    		</collision-->
+    </link>
   <gazebo reference="wall_1">
 	<material>Gazebo/White</material>
@@ -685,15 +663,15 @@
 	<selfCollide>false</selfCollide>
   </gazebo>
-  <gazebo reference="wall_21">
-	<material>Gazebo/White</material>
-	<selfCollide>false</selfCollide>
-  </gazebo>
+  <!--gazebo reference="wall_21">
+	<material>Gazebo/White</material>
+	<selfCollide>false</selfCollide>
+  </gazebo-->
   <gazebo reference="wall_22">
 	<material>Gazebo/White</material>
 	<selfCollide>false</selfCollide>
   </gazebo>
-  <gazebo reference="wall_23">
-	<material>Gazebo/White</material>
-	<selfCollide>false</selfCollide>
-  </gazebo>
+  <!--gazebo reference="wall_23">
+	<material>Gazebo/White</material>
+	<selfCollide>false</selfCollide>
+  </gazebo-->
 </robot>
